File: power_cutoff_unit/power_cutoff_unit.kicad_sch (KiCad schematic)
At the start: 152 parts, among them J1 Conn_01x02, J10 Conn_01x02, J11 Conn_01x02_Pin, J12 Conn_01x04, J13 Conn_01x04, J14 Conn_01x04, J15 Conn_01x02, J16 Conn_01x02, J17 Conn_01x03, J18 Conn_01x02, J19 Conn_01x03, J2 Conn_01x02, J20 Conn_01x03, J3 Conn_01x02, J4 Conn_01x02, J5 Conn_01x02, J6 Conn_01x02, J7 Conn_01x02, J8 Conn_01x02, J9 Conn_01x02, K1 T9GS1L14-5, K2 G5Q-1-DC5, K3 G5Q-1-DC5, Q1 SSM3K341R, Q2 SSM3K341R, Q3 SSM3K341R, Q4 SSM3K341R, Q5 BSS138, SW1 SW_Push, SW2 SW_DIP_x02, U1 LMZ14201H, U2 MIC4426, U3 MIC4426, U4 ADuM120N, U5 LMR50410Y3FQDBVRQ1, U6 MCP2562-E-SN, U7 STM32F303K8Tx

Commit message: 配置考え直す。
Parts:
- removed C11, C13, C15: 1000u, Capacitor_THT:CP_Radial_D16.0mm_P7.50mm, symbol Device:C_Polarized
- removed C7: 0.1uF, symbol Device:C
- removed C9: 10uF, symbol Device:C
- removed D15, D25, D26, D27: LED, symbol Device:LED
- removed J17: Conn_01x03, symbol Connector_Generic:Conn_01x03
- removed J5, J7, J9: Conn_01x02, Connector_AMASS:AMASS_XT30PW-M_1x02_P2.50mm_Horizontal, symbol Connector_Generic:Conn_01x02
- removed R32: 1K, symbol Device:R
- removed R47, R48: 10K, Resistor_SMD:R_0603_1608Metric, symbol Device:R
- added C7, C9: 470u, Capacitor_THT:CP_Radial_D12.5mm_P5.00mm, symbol Device:C_Polarized
- C1, C16, C17, C2, C20, C21, C23, C24, C27, C28, C29, C3, C30, C31, C32, C34: footprint (none) -> Capacitor_SMD:C_0402_1005Metric
- C12, C14, C22, C6, C8: footprint (none) -> Capacitor_SMD:C_0805_2012Metric
- C18, C19, C33: footprint (none) -> Capacitor_SMD:C_0603_1608Metric
- C25: value 10u -> 4.7u; footprint (none) -> Capacitor_SMD:C_0805_2012Metric
- C26: value 0.1u -> 4.7u; footprint (none) -> Capacitor_SMD:C_0805_2012Metric
- C4, C5: footprint (none) -> Capacitor_SMD:C_1210_3225Metric
- D1, D10, D12, D13, D14, D16, D18, D19, D2, D20, D21, D22, D23, D24, D3, D4, D6, D7, D9: footprint (none) -> LED_SMD:LED_0603_1608Metric
- D17: footprint (none) -> Diode_SMD:D_SOD-123F
- J1, J2, J3: footprint Connector_AMASS:AMASS_XT30PW-M_1x02_P2.50mm_Horizontal -> Connector_AMASS:AMASS_XT60IPW-M_1x03_P7.20mm_Horizontal
- J11: footprint (none) -> Connector_PinHeader_2.54mm:PinHeader_1x02_P2.54mm_Vertical
- J12, J13: footprint (none) -> Connector_JST:JST_XH_B4B-XH-A_1x04_P2.50mm_Vertical
- J18: footprint Connector_JST:JST_XH_S2B-XH-A_1x02_P2.50mm_Horizontal -> Connector_JST:JST_XH_B2B-XH-A_1x02_P2.50mm_Vertical
- J19, J20: footprint (none) -> Connector_JST:JST_XH_B3B-XH-A_1x03_P2.50mm_Vertical
- J4, J6, J8: footprint Connector_AMASS:AMASS_XT30PW-M_1x02_P2.50mm_Horizontal -> Connector_AMASS:AMASS_XT60PW-F_1x02_P7.20mm_Horizontal
- JP1, JP2, JP3: footprint (none) -> Jumper:SolderJumper-2_P1.3mm_Open_RoundedPad1.0x1.5mm
- K1: footprint (none) -> GN10RELAY:T9G
- K2, K3: footprint (none) -> GN10RELAY:G5Q-1
- R1, R10, R11, R12, R13, R14, R17, R18, R21, R22, R23, R26, R27, R28, R29, R3, R30, R31, R33, R34, R35, R36, R39, R4, R40, R41, R42, R43, R44, R6, R7, R8: footprint (none) -> Resistor_SMD:R_0603_1608Metric
- R16, R19, R2, R24, R5, R9: footprint (none) -> Resistor_SMD:R_0402_1005Metric
- R20, R25: footprint (none) -> Package_TO_SOT_THT:TO-220-2_Vertical
- R45, R46, R49: value 1K -> 10K
- SW2: footprint Button_Switch_SMD:SW_DIP_SPSTx02_Slide_Omron_A6H-2101_W6.15mm_P1.27mm -> (none)
Connections:
- net GND1: now also C7.2
- net GND2: now also C9.2
- net SW_1: now also R45.2
- net SW_2: now also R46.2
- net SW_3: now also R49.2
- net at C14.1, J8.2 (Pin_2), K3.2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: now also C9.1
- net at C12.1, J6.2 (Pin_2), K2.2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: now also C7.1
Other:
- moved on the sheet: BZ1, C1, C10, C12, C14, C16, C17, C18, C19, C2, C20, C21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

Commit message: 何したか覚えてないけど。
Parts:
- removed C14: 10uF, Capacitor_SMD:C_0805_2012Metric, symbol Device:C
- removed C17: 0.1u, Capacitor_SMD:C_0402_1005Metric, symbol Device:C
- removed C19: 4.7uF, Capacitor_SMD:C_0603_1608Metric, symbol Device:C
- removed C9: 470u, Capacitor_THT:CP_Radial_D12.5mm_P5.00mm, symbol Device:C_Polarized
- removed D1, D12, D13: LED, LED_SMD:LED_0603_1608Metric, symbol Device:LED
- removed D11: SS2040FL, Diode_SMD:D_SOD-123F, symbol Device:D
- removed J3: Conn_01x02, Connector_AMASS:AMASS_XT60IPW-M_1x03_P7.20mm_Horizontal, symbol Connector_Generic:Conn_01x02
- removed J8: Conn_01x02, Connector_AMASS:AMASS_XT60PW-F_1x02_P7.20mm_Horizontal, symbol Connector_Generic:Conn_01x02
- removed K3: G5Q-1-DC5, GN10RELAY:G5Q-1, symbol GN10RELAY:G5Q-1
- removed Q4: SSM3K341R, Package_TO_SOT_SMD:SOT-23_Handsoldering, symbol Device:Q_NMOS_GSD
- removed R22: 1K, Resistor_SMD:R_0603_1608Metric, symbol Device:R
- removed R23: 20K, Resistor_SMD:R_0603_1608Metric, symbol Device:R
- removed R24: 1K, Resistor_SMD:R_0402_1005Metric, symbol Device:R
- removed R25: 25, Package_TO_SOT_THT:TO-220-2_Vertical, symbol Device:R
- removed R26, R6: 4.7K, Resistor_SMD:R_0603_1608Metric, symbol Device:R
- removed U2, U3: MIC4426, symbol Driver_FET:MIC4426
- added C11: 0.1u, Capacitor_SMD:C_0402_1005Metric, symbol Device:C
- added D15: Blue, LED_SMD:LED_0603_1608Metric_Pad1.05x0.95mm_HandSolder, symbol Device:LED
- added R32: 1K, Resistor_SMD:R_0603_1608Metric, symbol Device:R
- added R47, R48: 10K, Resistor_SMD:R_0603_1608Metric, symbol Device:R
- added SW3: SW_DIP_x02, Button_Switch_SMD:SW_DIP_SPSTx02_Slide_Omron_A6H-2101_W6.15mm_P1.27mm, symbol Switch:SW_DIP_x02
- added U3: MIC4427, Package_SO:SOIC-8_3.9x4.9mm_P1.27mm, symbol Driver_FET:MIC4427
- added U8: MOUDLE-SEEEDUINO-XIAO-ESP32C3, RF_Module:MCU_Seeed_ESP32C3, symbol MOUDLE-SEEEDUINO-XIAO-ESP32C3:MOUDLE-SEEEDUINO-XIAO-ESP32C3
- J15, J16: footprint Connector_JST:JST_XH_S2B-XH-A_1x02_P2.50mm_Horizontal -> Connector_JST:JST_XH_B2B-XH-A_1x02_P2.50mm_Vertical
- L1: footprint (none) -> GN10:DEM2818C
- SW1: footprint (none) -> GN10:SKRPABE010
- SW2: footprint (none) -> Button_Switch_SMD:SW_DIP_SPSTx02_Slide_Omron_A6H-2101_W6.15mm_P1.27mm
- U1: footprint (none) -> GN10:LMZ14201H
Connections:
- net iso_RELAY_GATE_2 is gone; now on net iso_RELAY_GATE: R17.1
- net +3.3V: now also C11.1, SW3.1, SW3.2, U8.12 (3V3)
- net DIP1: now also R47.1, SW3.4, U8.4 (PA11_A3_D3); no longer SW2.4, U7.26 (PB3)
- net DIP2: now also R48.1, SW3.3, U8.5 (PA8_A4_D4_SDA); no longer SW2.3, U7.27 (PB4)
- net ENABLE: now also U8.3 (PA10_A2_D2)
- net GND: now also C11.2, D15.1 (K), R47.2, R48.2, U8.13 (GND)
- net GNDPWR: now also U3.3 (GND)
- net VDD: now also U3.6 (V+)
- net iso_DISCHARGE: now also U3.4 (IN_B)
- net iso_DISCHARGE_GATE: now also U3.5 (OUT_B)
- net iso_RELAY: now also U3.2 (IN_A)
- net iso_RELAY_GATE_1 renamed iso_RELAY_GATE
- net iso_RELAY_GATE: now also U3.7 (OUT_A)
- new net: R32.1, U8.2 (PA4_A1_D1)
- new net: D15.2 (A), R32.2
- new net ID_SW: SW2.3, U7.27 (PB4)
- new net MODE_SW: SW2.4, U7.26 (PB3)
- no-connect marks 4 -> 12
Other:
- note added: "POWER CUTTOFF 1"
- note added: "WIRELESS"
- note removed: "POWER_CUTTOFF_1"
- note removed: "POWER_CUTTOFF_3"
- moved on the sheet: BZ1, C1, C10, C12, C16, C18, C2, C20, C21, C22, C23, C24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

Commit message: 電圧書いた。配置きれいにした。
Parts:
- removed U8: MOUDLE-SEEEDUINO-XIAO-ESP32C3, RF_Module:MCU_Seeed_ESP32C3, symbol MOUDLE-SEEEDUINO-XIAO-ESP32C3:MOUDLE-SEEEDUINO-XIAO-ESP32C3
- added U2: MOUDLE-SEEEDUINO-XIAO-ESP32C3, MOUDLE14P-SMD-2.54-21X17.8MM, symbol MOUDLE-SEEEDUINO-XIAO-ESP32C3:MOUDLE-SEEEDUINO-XIAO-ESP32C3
Connections:
- net +3.3V: now also U2.12 (3V3)
- net DIP1: now also U2.4 (PA11_A3_D3)
- net DIP2: now also U2.5 (PA8_A4_D4_SDA)
- net ENABLE: now also U2.3 (PA10_A2_D2)
- net GND: now also U2.13 (GND)
- net at R32.1: now also U2.2 (PA4_A1_D1)
- net VDD renamed +5VA
Other:
- note added: "+BATT : 8 ~ 35V"
- note added: "POWER (LOGIC)"
- note added: "POWER CUTTOFF 2"
- note added: "VCC : 4 ~ 35V"
- note added: "Vdrive : 0 ~ 35V"
- note removed: "POWER_CUTTOFF_2"
- note removed: "POWER_LOGIC"
- moved on the sheet: BZ1, C1, C10, C11, C12, C16, C18, C2, C22, C23, C24, C25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

Commit message: PCBに入ったけどコンデンサの放電用抵抗を小さくしたい。
Parts:
- C1: value 0.022uF -> 0.022u
- C12: value 10uF -> 10u
- C18: value 4.7uF -> 4.7u
- C2: value 4700pF -> 4700p
- J1, J2: footprint Connector_AMASS:AMASS_XT60IPW-M_1x03_P7.20mm_Horizontal -> Connector_AMASS:AMASS_XT60PW-M_1x02_P7.20mm_Horizontal
- R15, R20: value 25 -> 30; footprint Package_TO_SOT_THT:TO-220-2_Vertical -> Package_TO_SOT_SMD:TO-263-2_TabPin1
- U2: footprint MOUDLE14P-SMD-2.54-21X17.8MM -> RF_Module:MCU_Seeed_ESP32C3
Other:
- note added: "MAX : 10A"
- note added: "MAX : 30A"
Changed lines of the file:
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@@
 		)
 	)
+	(text "MAX : 10A"
+		(exclude_from_sim no)
+		(at 371.856 123.698 0)
+		(effects
+			(font
+				(size 2.54 2.54)
+			)
+		)
+	)
+	(text "MAX : 30A"
+		(exclude_from_sim no)
+		(at 370.586 32.004 0)
+		(effects
+			(font
+				(size 2.54 2.54)
+			)
+		)
+	)
 	(text "Select mode."
 		(exclude_from_sim no)
@@
 			)
 		)
-		(property "Value" "0.022uF"
+		(property "Value" "0.022u"
 			(at 50.8 173.736 90)
 			(effects
@@
 			)
 		)
-		(property "Footprint" "Connector_AMASS:AMASS_XT60IPW-M_1x03_P7.20mm_Horizontal"
+		(property "Footprint" "Connector_AMASS:AMASS_XT60PW-M_1x02_P7.20mm_Horizontal"
 			(at 72.39 63.5 0)
 			(effects
@@
 			)
 		)
-		(property "Value" "25"
+		(property "Value" "30"
 			(at 304.8 135.89 90)
 			(effects
@@
 			)
 		)
-		(property "Footprint" "Package_TO_SOT_THT:TO-220-2_Vertical"
+		(property "Footprint" "Package_TO_SOT_SMD:TO-263-2_TabPin1"
 			(at 304.8 140.208 90)
 			(effects
@@
 			)
 		)
-		(property "Value" "4700pF"
+		(property "Value" "4700p"
 			(at 60.96 141.224 0)
 			(effects
@@
 			)
 		)
-		(property "Footprint" "Connector_AMASS:AMASS_XT60IPW-M_1x03_P7.20mm_Horizontal"
+		(property "Footprint" "Connector_AMASS:AMASS_XT60PW-M_1x02_P7.20mm_Horizontal"
 			(at 38.1 63.5 0)
 			(effects
@@
 			)
 		)
-		(property "Value" "10uF"
+		(property "Value" "10u"
 			(at 279.4 176.5299 0)
 			(effects
@@
 			)
 		)
-		(property "Value" "25"
+		(property "Value" "30"
 			(at 353.06 57.1499 0)
 			(effects
@@
 			)
 		)
-		(property "Footprint" "Package_TO_SOT_THT:TO-220-2_Vertical"
+		(property "Footprint" "Package_TO_SOT_SMD:TO-263-2_TabPin1"
 			(at 348.742 55.88 90)
 			(effects
@@
 			)
 		)
-		(property "Value" "4.7uF"
+		(property "Value" "4.7u"
 			(at 466.09 58.4199 0)
 			(effects
@@
 			)
 		)
-		(property "Footprint" "MOUDLE14P-SMD-2.54-21X17.8MM"
+		(property "Footprint" "RF_Module:MCU_Seeed_ESP32C3"
 			(at 410.21 303.53 0)
 			(effects

Commit message: 配置考え始めた
Parts:
- removed C11: 0.1u, Capacitor_SMD:C_0402_1005Metric, symbol Device:C
- removed C3: 1uF, Capacitor_SMD:C_0402_1005Metric, symbol Device:C
- removed J18: Conn_01x02, Connector_JST:JST_XH_B2B-XH-A_1x02_P2.50mm_Vertical, symbol Connector_Generic:Conn_01x02
- removed J19: Conn_01x03, Connector_JST:JST_XH_B3B-XH-A_1x03_P2.50mm_Vertical, symbol Connector_Generic:Conn_01x03
- removed R49: 10K, Resistor_SMD:R_0603_1608Metric, symbol Device:R
- J10: footprint Connector_AMASS:AMASS_XT30PW-M_1x02_P2.50mm_Horizontal -> Connector_AMASS:AMASS_XT30U-M_1x02_P5.0mm_Vertical
- R15: value 30 -> 50
- R3, R32, R4: footprint Resistor_SMD:R_0603_1608Metric -> Resistor_SMD:R_0402_1005Metric
Other:
- note removed: "Connect to remote emergency stop."
- moved on the sheet: C6, J15, J16, R45, R46

Commit message: PCBの配置考え中
Parts:
- J14: footprint Connector_JST:JST_XH_B4B-XH-A_1x04_P2.50mm_Vertical -> Connector_PinHeader_2.54mm:PinHeader_1x04_P2.54mm_Vertical
- J20: footprint Connector_JST:JST_XH_B3B-XH-A_1x03_P2.50mm_Vertical -> Connector_PinHeader_2.54mm:PinHeader_1x03_P2.54mm_Vertical
Changed lines of the file:
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@@
 			)
 		)
-		(property "Footprint" "Connector_JST:JST_XH_B4B-XH-A_1x04_P2.50mm_Vertical"
+		(property "Footprint" "Connector_PinHeader_2.54mm:PinHeader_1x04_P2.54mm_Vertical"
 			(at 509.27 313.69 0)
 			(effects
@@
 			)
 		)
-		(property "Footprint" "Connector_JST:JST_XH_B3B-XH-A_1x03_P2.50mm_Vertical"
+		(property "Footprint" "Connector_PinHeader_2.54mm:PinHeader_1x03_P2.54mm_Vertical"
 			(at 537.21 314.96 0)
 			(effects

Commit message: 高額だし、大きいので5Vラインのスイッチングレギュレーターを変更。
Parts:
- removed C1: 0.022u, Capacitor_SMD:C_0402_1005Metric, symbol Device:C
- removed C2: 4700p, Capacitor_SMD:C_0402_1005Metric, symbol Device:C
- removed C23: 1u, Capacitor_SMD:C_0402_1005Metric, symbol Device:C
- removed C25: 4.7u, Capacitor_SMD:C_0805_2012Metric, symbol Device:C
- removed C4, C5: 47uF, Capacitor_SMD:C_1210_3225Metric, symbol Device:C
- removed C6: 10uF, Capacitor_SMD:C_0805_2012Metric, symbol Device:C
- removed R1: 100K, Resistor_SMD:R_0603_1608Metric, symbol Device:R
- removed R2: 34K, Resistor_SMD:R_0402_1005Metric, symbol Device:R
- removed R3: 24K, Resistor_SMD:R_0402_1005Metric, symbol Device:R
- removed R4: 4.7K, Resistor_SMD:R_0402_1005Metric, symbol Device:R
- removed R5: 6.49K, Resistor_SMD:R_0402_1005Metric, symbol Device:R
- removed U1: LMZ14201H, GN10:LMZ14201H, symbol LMZ14201H:LMZ14201H
- added C11: 10u, Capacitor_SMD:C_0805_2012Metric, symbol Device:C
- added C3: 2.2u, Capacitor_SMD:C_0805_2012Metric, symbol Device:C
- added C9: 0.1u, Capacitor_SMD:C_0402_1005Metric, symbol Device:C
- added D1: SS2040FL, Diode_SMD:D_SOD-123F, symbol Device:D
- added L2: 4.7u, GN10:DEM2818C, symbol Device:L
- added U8: LMR50410Y5FQDBVRQ1, Package_TO_SOT_SMD:SOT-23-6, symbol GN10POWER:LMR50410
- C22: value 4.7u -> 2.2u
- C26: value 4.7u -> 10u
- L1: value 4.7u -> 3.3u
Connections:
- net +5VA: now also C11.1, D1.2 (A), L2.2, U8.3 (FB)
- net +BATT: now also C3.1, D1.1 (K), U8.4 (EN), U8.5 (VIN)
- net GNDPWR: now also C11.2, C3.2, U8.2 (GND)
- new net: C9.2, L2.1, U8.6 (SW)
- new net: C9.1, U8.1 (CB)
Other:
- moved on the sheet: C12, C16, C18, C7, D10, D8, D9, J6, K2, Q3, R17, R18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
