File: hardware/PowerCutoffBoard/PowerCutoffBoard.kicad_pcb (KiCad board)
At the start: 2 copper layers, 5 parts, among them U1 STM32G431CBUx, U2 MIC4427, U3 MCP2562-E-SN

Commit message: update: PowerCutoffBoard's schematic.
Parts:
- removed K1: ~, GN10_Parts:FBR562
- removed U1: STM32G431CBUx, Package_DFN_QFN:QFN-48-1EP_7x7mm_P0.5mm_EP5.6x5.6mm
- removed U2: MIC4427, Package_SO:SOIC-8_3.9x4.9mm_P1.27mm
- removed U3: MCP2562-E-SN, Package_SO:SOIC-8_3.9x4.9mm_P1.27mm
- removed U4: ~, GN10_Parts:LoRa-E5

Commit message: add: parts list. update: schematic.
Parts:
- added C19: 2700u, Capacitor_THT:CP_Radial_D18.0mm_P7.50mm, F.Cu at (130.5, 56.0)
- added C20: 2700u, Capacitor_THT:CP_Radial_D18.0mm_P7.50mm, F.Cu at (118.5, 56.0)
- added J5: XT30, Connector_AMASS:AMASS_XT30U-M_1x02_P5.0mm_Vertical, F.Cu at (156.5, 94.0)
- added J6: XT60, Connector_AMASS:AMASS_XT60-M_1x02_P7.20mm_Vertical, F.Cu at (111.4, 93.0)
- added J7: XT60, Connector_AMASS:AMASS_XT60-M_1x02_P7.20mm_Vertical, F.Cu at (138.6, 93.0)
- added J8: XT60, Connector_AMASS:AMASS_XT60-F_1x02_P7.20mm_Vertical, F.Cu at (111.4, 40.0)
- added J9: XT60, Connector_AMASS:AMASS_XT60-F_1x02_P7.20mm_Vertical, F.Cu at (137.6, 40.0)
- added K1: FBR562ND12-W, GN10_Parts:FBR562, F.Cu at (127.5, 79.0)
- added Q1: SSM3K341R, Package_TO_SOT_SMD:SOT-23, F.Cu at (151.9, 80.3)
- added Q2: SSM3K341R, Package_TO_SOT_SMD:SOT-23, F.Cu at (151.9, 85.0)
- added U1: STM32G431CBUx, Package_DFN_QFN:QFN-48-1EP_7x7mm_P0.5mm_EP5.6x5.6mm, F.Cu at (158.3, 56.9)
- added U2: MIC4427, Package_SO:SOIC-8_3.9x4.9mm_P1.27mm, F.Cu at (159.0, 83.0)
- added U3: MCP2562-E-SN, Package_SO:SOIC-8_3.9x4.9mm_P1.27mm, F.Cu at (172.0, 55.0)
- added U4: Wio-E5, GN10_Parts:LoRa-E5, F.Cu at (158.0, 42.0)
- added U5: OSL10326_IRA, GN10_Parts:OSL10326, F.Cu at (153.6, 71.0)
- added U6: 3.3V, Package_TO_SOT_SMD:SOT-223-3_TabPin2, F.Cu at (165.0, 69.0)

Commit message: update
Parts:
- added C1: 0.1u, Capacitor_SMD:C_0603_1608Metric_Pad1.08x0.95mm_HandSolder, F.Cu at (69.1, 48.8)
- added C10: 0.1u, Capacitor_SMD:C_0402_1005Metric_Pad0.74x0.62mm_HandSolder, F.Cu at (61.8, 90.0)
- added C11: 0.1u, Capacitor_SMD:C_0402_1005Metric_Pad0.74x0.62mm_HandSolder, F.Cu at (61.8, 92.0)
- added C12: 1u, Capacitor_SMD:C_0402_1005Metric_Pad0.74x0.62mm_HandSolder, F.Cu at (61.8, 93.9)
- added C13: 4.7u, Capacitor_SMD:C_0603_1608Metric_Pad1.08x0.95mm_HandSolder, F.Cu at (69.1, 63.8)
- added C14: 0.1u, Capacitor_SMD:C_0603_1608Metric_Pad1.08x0.95mm_HandSolder, F.Cu at (69.1, 66.3)
- added C15: 10u, Capacitor_SMD:C_0805_2012Metric_Pad1.18x1.45mm_HandSolder, F.Cu at (82.4, 33.5)
- added C16: 10u, Capacitor_SMD:C_0805_2012Metric_Pad1.18x1.45mm_HandSolder, F.Cu at (82.4, 36.5)
- added C17: 10u, Capacitor_SMD:C_0805_2012Metric_Pad1.18x1.45mm_HandSolder, F.Cu at (82.4, 39.5)
- added C18: 10u, Capacitor_SMD:C_0805_2012Metric_Pad1.18x1.45mm_HandSolder, F.Cu at (82.4, 42.5)
- added C2: 0.1u, Capacitor_SMD:C_0603_1608Metric_Pad1.08x0.95mm_HandSolder, F.Cu at (69.1, 51.3)
- added C21: 4.7u, Capacitor_SMD:C_0603_1608Metric_Pad1.08x0.95mm_HandSolder, F.Cu at (73.4, 48.8)
- added C22: 0.1u, Capacitor_SMD:C_0603_1608Metric_Pad1.08x0.95mm_HandSolder, F.Cu at (73.4, 51.3)
- added C3: 10u, Capacitor_SMD:C_0805_2012Metric_Pad1.18x1.45mm_HandSolder, F.Cu at (82.4, 27.5)
- added C4: 10u, Capacitor_SMD:C_0805_2012Metric_Pad1.18x1.45mm_HandSolder, F.Cu at (82.4, 30.5)
- added C5: 0.1u, Capacitor_SMD:C_0603_1608Metric_Pad1.08x0.95mm_HandSolder, F.Cu at (69.1, 53.8)
- added C6: 4.7u, Capacitor_SMD:C_0603_1608Metric_Pad1.08x0.95mm_HandSolder, F.Cu at (69.1, 56.3)
- added C7: 0.1u, Capacitor_SMD:C_0603_1608Metric_Pad1.08x0.95mm_HandSolder, F.Cu at (69.1, 58.8)
- added C8: 0.1u, Capacitor_SMD:C_0603_1608Metric_Pad1.08x0.95mm_HandSolder, F.Cu at (69.1, 61.3)
- added C9: 0.1u, Capacitor_SMD:C_0402_1005Metric_Pad0.74x0.62mm_HandSolder, F.Cu at (61.8, 88.0)
- added D10: LED, LED_SMD:LED_0603_1608Metric_Pad1.05x0.95mm_HandSolder, F.Cu at (37.1, 86.4)
- added D11: LED, LED_SMD:LED_0603_1608Metric_Pad1.05x0.95mm_HandSolder, F.Cu at (37.1, 89.0)
- added D12: D, Diode_SMD:D_SOD-123, F.Cu at (74.8, 91.8)
- added D13: LED, LED_SMD:LED_0603_1608Metric_Pad1.05x0.95mm_HandSolder, F.Cu at (37.1, 91.6)
- added D3: D, Diode_SMD:D_SMA_Handsoldering, B.Cu at (29.0, 147.0)
- added D4: D, Diode_SMD:D_SMA_Handsoldering, B.Cu at (42.0, 147.0)
- added D5: LED, LED_SMD:LED_0603_1608Metric_Pad1.05x0.95mm_HandSolder, F.Cu at (37.1, 73.4)
- added D6: LED, LED_SMD:LED_0603_1608Metric_Pad1.05x0.95mm_HandSolder, F.Cu at (37.1, 76.0)
- added D7: LED, LED_SMD:LED_0603_1608Metric_Pad1.05x0.95mm_HandSolder, F.Cu at (37.1, 78.6)
- added D8: LED, LED_SMD:LED_0603_1608Metric_Pad1.05x0.95mm_HandSolder, F.Cu at (37.1, 81.2)
- added D9: LED, LED_SMD:LED_0603_1608Metric_Pad1.05x0.95mm_HandSolder, F.Cu at (37.1, 83.8)
- added J1: Conn_01x04, Connector_JST:JST_XH_B4B-XH-A_1x04_P2.50mm_Vertical, F.Cu at (55.9, 50.9)
- added J11: Conn_Coaxial, Connector_Coaxial:SMA_Molex_73251-2120_EdgeMount_Horizontal, F.Cu at (19.3, 70.9)
- added J2: Conn_01x04, Connector_JST:JST_XH_B4B-XH-A_1x04_P2.50mm_Vertical, F.Cu at (55.9, 58.7)
- added J3: Conn_01x04, Connector_JST:JST_XH_B4B-XH-A_1x04_P2.50mm_Vertical, F.Cu at (55.9, 66.5)
- added J4: Conn_01x04, Connector_JST:JST_XH_B4B-XH-A_1x04_P2.50mm_Vertical, F.Cu at (55.9, 74.3)
- added R1: 50, Resistor_SMD:R_2010_5025Metric_Pad1.40x2.65mm_HandSolder, F.Cu at (19.0, 155.0)
- added R10: 1k, Capacitor_SMD:C_0603_1608Metric_Pad1.08x0.95mm_HandSolder, F.Cu at (77.8, 51.3)
- added R11: 1k, Capacitor_SMD:C_0603_1608Metric_Pad1.08x0.95mm_HandSolder, F.Cu at (77.8, 53.8)
- added R12: 1k, Capacitor_SMD:C_0603_1608Metric_Pad1.08x0.95mm_HandSolder, F.Cu at (77.8, 56.3)
- added R13: 1k, Capacitor_SMD:C_0603_1608Metric_Pad1.08x0.95mm_HandSolder, F.Cu at (77.8, 58.8)
- added R14: 1k, Capacitor_SMD:C_0603_1608Metric_Pad1.08x0.95mm_HandSolder, F.Cu at (77.8, 61.3)
- added R15: 1k, Capacitor_SMD:C_0603_1608Metric_Pad1.08x0.95mm_HandSolder, F.Cu at (77.8, 63.8)
- added R16: 1k, Capacitor_SMD:C_0603_1608Metric_Pad1.08x0.95mm_HandSolder, F.Cu at (77.8, 66.3)
- added R17: 1k, Capacitor_SMD:C_0603_1608Metric_Pad1.08x0.95mm_HandSolder, F.Cu at (82.1, 48.8)
- added R18: 1k, Capacitor_SMD:C_0603_1608Metric_Pad1.08x0.95mm_HandSolder, F.Cu at (82.1, 51.3)
- added R19: 1k, Capacitor_SMD:C_0603_1608Metric_Pad1.08x0.95mm_HandSolder, F.Cu at (82.1, 53.8)
- added R2: 50, Resistor_SMD:R_2010_5025Metric_Pad1.40x2.65mm_HandSolder, F.Cu at (53.0, 155.0)
- added R20: 470, Capacitor_SMD:C_0603_1608Metric_Pad1.08x0.95mm_HandSolder, F.Cu at (82.1, 56.3)
- added R21: 1k, Capacitor_SMD:C_0603_1608Metric_Pad1.08x0.95mm_HandSolder, F.Cu at (82.1, 58.8)
- added R5: 1k, Capacitor_SMD:C_0603_1608Metric_Pad1.08x0.95mm_HandSolder, F.Cu at (73.4, 58.8)
- added R6: 1k, Capacitor_SMD:C_0603_1608Metric_Pad1.08x0.95mm_HandSolder, F.Cu at (73.4, 61.3)
- added R7: 1k, Capacitor_SMD:C_0603_1608Metric_Pad1.08x0.95mm_HandSolder, F.Cu at (73.4, 63.8)
- added R8: 1k, Capacitor_SMD:C_0603_1608Metric_Pad1.08x0.95mm_HandSolder, F.Cu at (73.4, 66.3)
- added R9: 1k, Capacitor_SMD:C_0603_1608Metric_Pad1.08x0.95mm_HandSolder, F.Cu at (77.8, 48.8)
- added SW1: SW_Push, GN10_Parts:TVAF, F.Cu at (18.8, 79.3)
- added SW2: SW_Push, GN10_Parts:TVAF, F.Cu at (18.8, 84.4)
- added SW3: SW_Push, GN10_Parts:TVAF, F.Cu at (18.8, 89.4)
- added TP1: TestPoint, TestPoint:TestPoint_Pad_D1.0mm, F.Cu at (49.4, 81.7)
- added TP2: TestPoint, TestPoint:TestPoint_Pad_D1.0mm, F.Cu at (49.4, 84.7)
- added TP3: TestPoint, TestPoint:TestPoint_Pad_D1.0mm, F.Cu at (49.4, 87.8)
- added TP4: TestPoint, TestPoint:TestPoint_Pad_D1.0mm, F.Cu at (49.4, 90.8)
- added Y1: Crystal_GND2, Crystal:Resonator_SMD_Murata_CSTxExxV-3Pin_3.0x1.1mm_HandSoldering, F.Cu at (69.5, 92.5)
- moved U1 135.0 mm to (27.5, 90.5)
- moved U3 130.3 mm to (43.5, 76.9)
- moved J9 120.7 mm to (42.2, 114.0), turned to 0 degrees
- moved C20 120.6 mm to (22.5, 129.0), turned to 0 degrees
- moved U2 116.2 mm to (43.5, 70.3)
- moved K1 116.0 mm to (35.8, 150.0)
- moved J6 115.3 mm to (21.4, 165.0)
- moved J7 115.3 mm to (48.6, 165.0)
- moved U5 111.1 mm to (43.6, 86.4)
- moved J8 110.4 mm to (29.4, 114.0), turned to 180 degrees
- moved C19 109.1 mm to (49.5, 129.0), turned to 180 degrees
- moved U6 108.5 mm to (57.4, 82.9)
- moved U4 89.6 mm to (74.8, 75.2)
- moved J5 86.3 mm to (70.5, 86.5), turned to 0 degrees
- moved Q1 70.5 mm to (81.6, 85.3)
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