File: hardware/PowerCutoffBoard/PowerCutoffBoard.kicad_sch (KiCad schematic)
At the start: 80 parts, among them J1 Conn_01x04, J10 Conn_01x04, J2 Conn_01x04, J3 Conn_01x04, J4 Conn_01x04, J5 XT30, J6 XT60, J7 XT60, J8 XT60, J9 XT60, K1 FBR562ND12-W, Q1 SSM3K341R, Q2 SSM3K341R, SW1 SW_Push, SW2 SW_Push, SW3 SW_Push, U1 STM32G431CBUx, U2 MIC4427, U3 MCP2562-E-SN, U4 Wio-E5, U5 OSL10326_IRA, U6 3.3V, Y1 Crystal_GND2

Commit message: add: parts list. update: schematic.
Parts:
- C19, C20: value 4700u -> 2700u; footprint (none) -> Capacitor_THT:CP_Radial_D18.0mm_P7.50mm
- J5: footprint (none) -> Connector_AMASS:AMASS_XT30U-M_1x02_P5.0mm_Vertical
- J6, J7: footprint (none) -> Connector_AMASS:AMASS_XT60-M_1x02_P7.20mm_Vertical
- J8, J9: footprint (none) -> Connector_AMASS:AMASS_XT60-F_1x02_P7.20mm_Vertical
- Q1, Q2: footprint (none) -> Package_TO_SOT_SMD:SOT-23
Other:
- moved on the sheet: C19, C20
Changed lines of the file:
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@@
 	)
 	(junction
-		(at 363.22 73.66)
+		(at 368.3 73.66)
 		(diameter 0)
 		(color 0 0 0 0)
@@
 	)
 	(junction
-		(at 363.22 66.04)
+		(at 368.3 66.04)
 		(diameter 0)
 		(color 0 0 0 0)
@@
 	)
 	(junction
-		(at 363.22 40.64)
+		(at 368.3 40.64)
 		(diameter 0)
 		(color 0 0 0 0)
 	)
 	(junction
-		(at 363.22 48.26)
+		(at 368.3 48.26)
 		(diameter 0)
 		(color 0 0 0 0)
@@
 	(wire
 		(pts
-			(xy 355.6 66.04) (xy 363.22 66.04)
+			(xy 360.68 66.04) (xy 368.3 66.04)
 		)
 		(stroke
@@
 	(wire
 		(pts
-			(xy 54.61 139.7) (xy 62.23 139.7)
+			(xy 368.3 40.64) (xy 378.46 40.64)
 		)
 		(stroke
@@
 	(wire
 		(pts
-			(xy 24.13 223.52) (xy 38.1 223.52)
+			(xy 54.61 139.7) (xy 62.23 139.7)
 		)
 		(stroke
@@
 	(wire
 		(pts
-			(xy 320.04 133.35) (xy 334.01 133.35)
+			(xy 24.13 223.52) (xy 38.1 223.52)
 		)
 		(stroke
@@
 	(wire
 		(pts
-			(xy 110.49 54.61) (xy 110.49 53.34)
+			(xy 320.04 133.35) (xy 334.01 133.35)
 		)
 		(stroke
@@
 	(wire
 		(pts
-			(xy 269.24 264.16) (xy 271.78 264.16)
+			(xy 110.49 54.61) (xy 110.49 53.34)
 		)
 		(stroke
@@
 	(wire
 		(pts
-			(xy 269.24 251.46) (xy 271.78 251.46)
+			(xy 269.24 264.16) (xy 271.78 264.16)
 		)
 		(stroke
@@
 	(wire
 		(pts
-			(xy 299.72 82.55) (xy 299.72 83.82)
+			(xy 269.24 251.46) (xy 271.78 251.46)
 		)
 		(stroke
@@
 	(wire
 		(pts
-			(xy 363.22 40.64) (xy 378.46 40.64)
+			(xy 299.72 82.55) (xy 299.72 83.82)
 		)
 		(stroke
@@
 	(wire
 		(pts
-			(xy 355.6 40.64) (xy 363.22 40.64)
+			(xy 360.68 40.64) (xy 368.3 40.64)
 		)
 		(stroke
@@
 	(wire
 		(pts
-			(xy 363.22 73.66) (xy 378.46 73.66)
+			(xy 368.3 73.66) (xy 378.46 73.66)
 		)
 		(stroke
@@
 	(wire
 		(pts
-			(xy 363.22 50.8) (xy 363.22 48.26)
+			(xy 368.3 50.8) (xy 368.3 48.26)
 		)
 		(stroke
@@
 	(wire
 		(pts
-			(xy 261.62 46.99) (xy 261.62 49.53)
+			(xy 368.3 66.04) (xy 378.46 66.04)
 		)
 		(stroke
@@
 	(wire
 		(pts
-			(xy 87.63 120.65) (xy 87.63 128.27)
+			(xy 261.62 46.99) (xy 261.62 49.53)
 		)
 		(stroke
@@
 	(wire
 		(pts
-			(xy 236.22 57.15) (xy 248.92 57.15)
+			(xy 87.63 120.65) (xy 87.63 128.27)
 		)
 		(stroke
@@
 	(wire
 		(pts
-			(xy 363.22 66.04) (xy 378.46 66.04)
+			(xy 236.22 57.15) (xy 248.92 57.15)
 		)
 		(stroke
@@
 	(wire
 		(pts
-			(xy 363.22 48.26) (xy 378.46 48.26)
-		)
-		(stroke
-			(width 0)
-			(type default)
-		)
-	)
-	(wire
-		(pts
 			(xy 41.91 182.88) (xy 25.4 182.88)
 		)
@@
 	(wire
 		(pts
-			(xy 363.22 76.2) (xy 363.22 73.66)
+			(xy 368.3 76.2) (xy 368.3 73.66)
 		)
 		(stroke
@@
 	(wire
 		(pts
+			(xy 368.3 48.26) (xy 378.46 48.26)
+		)
+		(stroke
+			(width 0)
+			(type default)
+		)
+	)
+	(wire
+		(pts
 			(xy 337.82 204.47) (xy 350.52 204.47)
 		)
@@
 	(global_label "OUTPUT_A"
 		(shape input)
-		(at 355.6 40.64 180)
+		(at 360.68 40.64 180)
 		(fields_autoplaced yes)
 		(effects
@@
 		)
 		(property "Intersheetrefs" "${INTERSHEET_REFS}"
-			(at 343.3619 40.64 0)
+			(at 348.4419 40.64 0)
 			(effects
 				(font
@@
 	(global_label "OUTPUT_B"
 		(shape input)
-		(at 355.6 66.04 180)
+		(at 360.68 66.04 180)
 		(fields_autoplaced yes)
 		(effects
@@
 		)
 		(property "Intersheetrefs" "${INTERSHEET_REFS}"
-			(at 343.1805 66.04 0)
+			(at 348.2605 66.04 0)
 			(effects
 				(font
@@
 	(symbol
 		(lib_id "power:GNDPWR")
-		(at 363.22 76.2 0)
+		(at 368.3 76.2 0)
 		(unit 1)
 		(exclude_from_sim no)
@@
 		(fields_autoplaced yes)
 		(property "Reference" "#PWR051"
-			(at 363.22 81.28 0)
+			(at 368.3 81.28 0)
 			(effects
 				(font
@@
 		)
 		(property "Value" "GNDPWR"
-			(at 363.093 80.01 0)
+			(at 368.173 80.01 0)
 			(effects
 				(font
@@
 		)
 		(property "Footprint" ""
-			(at 363.22 77.47 0)
+			(at 368.3 77.47 0)
 			(effects
 				(font
@@
 		)
 		(property "Datasheet" ""
-			(at 363.22 77.47 0)
+			(at 368.3 77.47 0)
 			(effects
 				(font
@@
 		)
 		(property "Description" "Power symbol creates a global label with name \"GNDPWR\" , global ground"
-			(at 363.22 76.2 0)
+			(at 368.3 76.2 0)
 			(effects
 				(font
@@
 	(symbol
 		(lib_id "Device:C_Polarized")
-		(at 363.22 44.45 0)
+		(at 368.3 44.45 0)
 		(unit 1)
 		(exclude_from_sim no)
@@
 		(fields_autoplaced yes)
 		(property "Reference" "C20"
-			(at 367.03 42.2909 0)
+			(at 372.11 42.2909 0)
 			(effects
 				(font
@@
 			)
 		)
-		(property "Value" "4700u"
-			(at 367.03 44.8309 0)
+		(property "Value" "2700u"
+			(at 372.11 44.8309 0)
 			(effects
 				(font
@@
 			)
 		)
-		(property "Footprint" ""
-			(at 364.1852 48.26 0)
+		(property "Footprint" "Capacitor_THT:CP_Radial_D18.0mm_P7.50mm"
+			(at 369.2652 48.26 0)
 			(effects
 				(font
@@
 		)
 		(property "Datasheet" "~"
-			(at 363.22 44.45 0)
+			(at 368.3 44.45 0)
 			(effects
 				(font
@@
 		)
 		(property "Description" "Polarized capacitor"
-			(at 363.22 44.45 0)
+			(at 368.3 44.45 0)
 			(effects
 				(font
@@
 			)
 		)
-		(property "Footprint" ""
+		(property "Footprint" "Package_TO_SOT_SMD:SOT-23"
 			(at 264.16 68.58 0)
 			(effects
@@
 			)
 		)
-		(property "Footprint" ""
+		(property "Footprint" "Connector_AMASS:AMASS_XT30U-M_1x02_P5.0mm_Vertical"
 			(at 33.02 137.16 0)
 			(effects
@@
 			)
 		)
-		(property "Footprint" ""
+		(property "Footprint" "Connector_AMASS:AMASS_XT60-F_1x02_P7.20mm_Vertical"
 			(at 384.81 69.85 0)
 			(effects
@@
 	(symbol
 		(lib_id "power:GNDPWR")
-		(at 363.22 50.8 0)
+		(at 368.3 50.8 0)
 		(unit 1)
 		(exclude_from_sim no)
@@
 		(fields_autoplaced yes)
 		(property "Reference" "#PWR050"
-			(at 363.22 55.88 0)
+			(at 368.3 55.88 0)
 			(effects
 				(font
@@
 		)
 		(property "Value" "GNDPWR"
-			(at 363.093 54.61 0)
+			(at 368.173 54.61 0)
 			(effects
 				(font
@@
 		)
 		(property "Footprint" ""
-			(at 363.22 52.07 0)
+			(at 368.3 52.07 0)
 			(effects
 				(font
@@
 		)
 		(property "Datasheet" ""
-			(at 363.22 52.07 0)
+			(at 368.3 52.07 0)
 			(effects
 				(font
@@
 		)
 		(property "Description" "Power symbol creates a global label with name \"GNDPWR\" , global ground"
-			(at 363.22 50.8 0)
+			(at 368.3 50.8 0)
 			(effects
 				(font
@@
 	(symbol
 		(lib_id "Device:C_Polarized")
-		(at 363.22 69.85 0)
+		(at 368.3 69.85 0)
 		(unit 1)
 		(exclude_from_sim no)
@@
 		(fields_autoplaced yes)
 		(property "Reference" "C19"
-			(at 367.03 67.6909 0)
+			(at 372.11 67.6909 0)
 			(effects
 				(font
@@
 			)
 		)
-		(property "Value" "4700u"
-			(at 367.03 70.2309 0)
+		(property "Value" "2700u"
+			(at 372.11 70.2309 0)
 			(effects
 				(font
@@
 			)
 		)
-		(property "Footprint" ""
-			(at 364.1852 73.66 0)
+		(property "Footprint" "Capacitor_THT:CP_Radial_D18.0mm_P7.50mm"
+			(at 369.2652 73.66 0)
 			(effects
 				(font
@@
 		)
 		(property "Datasheet" "~"
-			(at 363.22 69.85 0)
+			(at 368.3 69.85 0)
 			(effects
 				(font
@@
 		)
 		(property "Description" "Polarized capacitor"
-			(at 363.22 69.85 0)
+			(at 368.3 69.85 0)
 			(effects
 				(font
@@
 			)
 		)
-		(property "Footprint" ""
+		(property "Footprint" "Connector_AMASS:AMASS_XT60-M_1x02_P7.20mm_Vertical"
 			(at 104.14 49.53 0)
 			(effects
@@
 			)
 		)
-		(property "Footprint" ""
+		(property "Footprint" "Connector_AMASS:AMASS_XT60-M_1x02_P7.20mm_Vertical"
 			(at 104.14 74.93 0)
 			(effects
@@
 			)
 		)
-		(property "Footprint" ""
+		(property "Footprint" "Connector_AMASS:AMASS_XT60-F_1x02_P7.20mm_Vertical"
 			(at 384.81 44.45 0)
 			(effects
@@
 			)
 		)
-		(property "Footprint" ""
+		(property "Footprint" "Package_TO_SOT_SMD:SOT-23"
 			(at 175.26 68.58 0)
 			(effects

Commit message: update
Parts:
- removed AE1: Antenna, symbol Device:Antenna
- removed D1, D2: Red, symbol Device:LED
- removed J10: Conn_01x04, symbol Connector_Generic:Conn_01x04
- removed R3, R4: 1k, symbol Device:R
- added J11: Conn_Coaxial, Connector_Coaxial:SMA_Molex_73251-2120_EdgeMount_Horizontal, symbol Connector:Conn_Coaxial
- added TP1, TP2, TP3, TP4: TestPoint, TestPoint:TestPoint_Pad_D1.0mm, symbol Connector:TestPoint
- C1, C13, C14, C2, C21, C22, C5, C6, C7, C8, R10, R11, R12, R13, R14, R15, R16, R17, R18, R19, R20, R21, R5, R6, R7, R8, R9: footprint (none) -> Capacitor_SMD:C_0603_1608Metric_Pad1.08x0.95mm_HandSolder
- C10, C11, C12, C9: footprint (none) -> Capacitor_SMD:C_0402_1005Metric_Pad0.74x0.62mm_HandSolder
- C15, C16, C17, C18, C3, C4: footprint (none) -> Capacitor_SMD:C_0805_2012Metric_Pad1.18x1.45mm_HandSolder
- D10, D11, D13, D5, D6, D7, D8, D9: footprint (none) -> LED_SMD:LED_0603_1608Metric_Pad1.05x0.95mm_HandSolder
- D12: footprint (none) -> Diode_SMD:D_SOD-123
- D3, D4: footprint (none) -> Diode_SMD:D_SMA_Handsoldering
- J1, J2, J3, J4: footprint (none) -> Connector_JST:JST_XH_B4B-XH-A_1x04_P2.50mm_Vertical
- R1, R2: footprint (none) -> Resistor_SMD:R_2010_5025Metric_Pad1.40x2.65mm_HandSolder
- SW1, SW2, SW3: footprint (none) -> GN10_Parts:TVAF
- Y1: footprint (none) -> Crystal:Resonator_SMD_Murata_CSTxExxV-3Pin_3.0x1.1mm_HandSoldering
Connections:
- net +3.3V: now also TP1.1
- net GND: now also J11.2 (Ext), TP3.1
- net LoRa_SWCLK: now also TP2.1
- net LoRa_SWDIO: now also TP4.1
- net at U4.15 (RFIO): now also J11.1 (In)
Other:
- moved on the sheet: C15, C16, C7, C8, J3, J4, U3
