File: hardware/PowerCutoffBoard2/PowerCutoffBoard2.kicad_pcb (KiCad board)
At the start: 2 copper layers, 19 parts, among them J2 Conn_01x03, J5 XT30, J6 XT60, J7 XT60, J8 XT60, J9 XT60, K1 FBR562ND12-W, Q1 SSM3K341R, Q2 SSM3K341R

Commit message: update
Parts:
- removed C1: 0.1u, Capacitor_SMD:C_0603_1608Metric_Pad1.08x0.95mm_HandSolder
- removed C3: 10u, Capacitor_SMD:C_0805_2012Metric_Pad1.18x1.45mm_HandSolder
- added R3: 24k, Resistor_SMD:R_0603_1608Metric_Pad0.98x0.95mm_HandSolder, B.Cu at (175.0, 103.5)
- added R4: 24k, Resistor_SMD:R_0603_1608Metric_Pad0.98x0.95mm_HandSolder, B.Cu at (175.0, 107.0)
- added REF**: MountingHole_3.2mm_M3, MountingHole:MountingHole_3.2mm_M3, F.Cu at (103.5, 88.5)
- added REF**: MountingHole_3.2mm_M3, MountingHole:MountingHole_3.2mm_M3, F.Cu at (181.5, 146.5)
- added REF**: MountingHole_3.2mm_M3, MountingHole:MountingHole_3.2mm_M3, F.Cu at (103.5, 146.5)
- added REF**: MountingHole_3.2mm_M3, MountingHole:MountingHole_3.2mm_M3, F.Cu at (181.5, 88.5)
- C2, C4: moved to B.Cu
- J5: footprint Connector_AMASS:AMASS_XT30U-M_1x02_P5.0mm_Vertical -> Connector_AMASS:AMASS_XT30PW-M_1x02_P2.50mm_Horizontal
- moved J2 124.0 mm to (171.3, 99.3), turned to -90 degrees
- moved Q1 117.7 mm to (175.8, 130.4), turned to 180 degrees
- moved Q2 117.6 mm to (175.8, 135.4), turned to 180 degrees
- moved J5 108.1 mm to (171.4, 122.7), turned to -90 degrees
- moved C4 106.0 mm to (166.0, 120.7), turned to 90 degrees
- moved J9 104.9 mm to (144.6, 90.8), turned to 180 degrees
- moved C2 103.3 mm to (168.0, 120.7), turned to 90 degrees
- moved C20 101.8 mm to (121.7, 106.0), turned to 180 degrees
- moved R2 98.0 mm to (148.7, 134.0)
- moved D3 97.8 mm to (124.6, 126.3)
- moved D4 97.5 mm to (137.3, 126.3)
- moved K1 97.4 mm to (130.9, 128.9)
- moved J7 97.0 mm to (143.3, 144.1)
- moved R1 96.5 mm to (113.1, 134.0)
- moved J6 95.7 mm to (114.8, 144.1)
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Connections:
- C19 pad 2: GNDPWR -> GNDD
- J7 pad 1: GNDPWR -> GNDD
- J9 pad 1: GNDPWR -> GNDD
- R2 pad 2: GNDPWR -> GNDD
Routing:
- net +12V: track 0.00 -> 66.6 mm
- net Net-(D3-A): track 0.00 -> 50.7 mm, vias 0 -> 1
- net Net-(D4-A): track 0.00 -> 39.8 mm, vias 0 -> 1
- net GATE_B: track 0.00 -> 36.7 mm
- net GATE_A: track 0.00 -> 36.2 mm
- net Net-(K1A-N.C.): track 0.00 -> 15.4 mm
- net Net-(K1B-N.C.): track 0.00 -> 5.22 mm
- added copper zone on B.Cu, net GND
- added copper zone on F.Cu, net GND
- added copper zone on B.Cu, net GNDD
- added copper zone on F.Cu, net GNDD
- added copper zone on B.Cu, net GNDPWR
- added copper zone on F.Cu, net GNDPWR
- added copper zone on B.Cu, net INPUT_A
- added copper zone on F.Cu, net INPUT_A
- added copper zone on B.Cu, net INPUT_B
- added copper zone on F.Cu, net INPUT_B
- added copper zone on B.Cu, net OUTPUT_A
- added copper zone on F.Cu, net OUTPUT_A
- added copper zone on B.Cu, net OUTPUT_B
- added copper zone on F.Cu, net OUTPUT_B
Other:
- board outline added: 85 x 65 mm

Commit message: generate: gaber PowerCutoffBoard2
Routing:
- net OUTPUT_B: vias 0 -> 38
- net OUTPUT_A: vias 0 -> 25
- net INPUT_B: vias 0 -> 14
- net INPUT_A: vias 0 -> 13
- net GNDPWR: vias 0 -> 72
- net GNDD: vias 0 -> 68
- net GND: vias 0 -> 57
Other:
- board text added: "Designed by: GN10/Gento Aiba"
- board text added: "PowerCutoffBoard-2"
- board text added: "https://github.com/ararobo/GN10RemoteEmergencyStop"
