File: hardware/RemoteSwitchBoard/RemoteSwitchBoard.kicad_sch (KiCad schematic)
At the start: 0 parts

Commit message: RemoteSwitchBoard sch
Parts:
- added BZ1: Buzzer, symbol Device:Buzzer
- added C1, C2, C4, C6: 0.1u, Capacitor_SMD:C_0603_1608Metric_Pad1.08x0.95mm_HandSolder, symbol Device:C
- added C3, C5: 4.7u, Capacitor_SMD:C_0603_1608Metric_Pad1.08x0.95mm_HandSolder, symbol Device:C
- added C7, C8: 10u, Capacitor_SMD:C_0603_1608Metric_Pad1.08x0.95mm_HandSolder, symbol Device:C
- added D1: D, Diode_SMD:Nexperia_CFP3_SOD-123W, symbol Device:D
- added D2, D4, D5, D6, D7, D9: LED, LED_SMD:LED_0603_1608Metric_Pad1.05x0.95mm_HandSolder, symbol Device:LED
- added H1, H2, H3, H4: MountingHole, MountingHole:MountingHole_3.2mm_M3, symbol Mechanical:MountingHole
- added J1: Conn_Coaxial, Connector_Coaxial:SMA_Molex_73251-2120_EdgeMount_Horizontal, symbol Connector:Conn_Coaxial
- added J2, J8: Conn_01x05, symbol Connector_Generic:Conn_01x05
- added J3, J4, J7: Conn_01x02, symbol Connector_Generic:Conn_01x02
- added J5, J6: Conn_01x04, Connector_JST:JST_XH_B4B-XH-A_1x04_P2.50mm_Vertical, symbol Connector_Generic:Conn_01x04
- added R1: 10k, Capacitor_SMD:C_0603_1608Metric_Pad1.08x0.95mm_HandSolder, symbol Device:R
- added R10, R11, R12, R13, R14, R2, R3, R4, R5, R6, R7, R9: 1k, Capacitor_SMD:C_0603_1608Metric_Pad1.08x0.95mm_HandSolder, symbol Device:R
- added SW1, SW2: SW_Push, GN10_Parts:TVAF, symbol Switch:SW_Push
- added TP1, TP2, TP3: TestPoint, TestPoint:TestPoint_Pad_D1.5mm, symbol Connector:TestPoint
- added U1: STM32F303K8Tx, Package_QFP:LQFP-32_7x7mm_P0.8mm, symbol MCU_ST_STM32F3:STM32F303K8Tx
- added U2: Wio-E5, GN10_Parts:LoRa-E5, symbol LoRa-E5:LoRa-E5
- added U3: 3.3V, Package_TO_SOT_SMD:SOT-223-3_TabPin2, symbol GN10_Parts:TPS1117LV33S
- added Y1: Crystal_GND2, Crystal:Resonator_SMD_Murata_CSTxExxV-3Pin_3.0x1.1mm_HandSoldering, symbol Device:Crystal_GND2
Connections:
- new net: J1.1 (In), U2.15 (RFIO)
- new net: D7.2 (A), R7.2
- new net: D6.2 (A), R6.2
- new net: D9.2 (A), R9.2
- new net: J7.1 (Pin_1), R14.2
- new net: D2.2 (A), R2.2
- new net: BZ1.1 (+), U1.6 (PA0)
- new net: U1.2 (PF0), Y1.1
- new net: U1.3 (PF1), Y1.3
- new net: J2.1 (Pin_1), R3.2
- new net: J2.4 (Pin_4), R12.2
- new net: D4.2 (A), R4.2
- new net: J2.2 (Pin_2), R10.2
- new net: J2.3 (Pin_3), R11.2
- new net: R1.1, U1.31 (BOOT0)
- new net: J3.1 (Pin_1), R13.2
- new net: D5.2 (A), R5.2
- new net +3.3V: C1.1, C2.1, C3.1, C5.1, C8.1, D1.2 (A), J4.2 (Pin_2), J5.1 (Pin_1), J6.2 (Pin_2), J8.5 (Pin_5), R2.1, R4.1, U1.1 (VDD), U1.17 (VDD), U1.5 (VDDA), U2.1 (VCC), U3.2 (VOUT)
- new net +5V: C7.1, D1.1 (K), U3.3 (VIN)
- new net DIP_1: J8.1 (Pin_1), U1.28 (PB5)
- new net DIP_2: J8.2 (Pin_2), U1.27 (PB4)
- new net DIP_3: J8.3 (Pin_3), U1.26 (PB3)
- new net DIP_4: J8.4 (Pin_4), U1.25 (PA15)
- new net GND: BZ1.2 (-), C1.2, C2.2, C3.2, C4.2, C5.2, C6.2, C7.2, C8.2, D4.1 (K), D5.1 (K), D6.1 (K), D7.1 (K), D9.1 (K), J1.2 (Ext), J2.5 (Pin_5), J3.2 (Pin_2), J5.3 (Pin_3), J6.4 (Pin_4), J7.2 (Pin_2), R1.2, SW1.1, SW2.1, U1.16 (VSS), U1.32 (VSS), U2.14 (GND), U2.16 (GND), U2.2 (GND), U2.22 (GND), U3.1 (GND), Y1.2
- new net LED_1: R14.1, U1.12 (PA6)
- new net LED_2: R9.1, U1.11 (PA5)
- new net LED_3: R3.1, U1.10 (PA4)
- new net LED_4: R10.1, U1.18 (PA8)
- new net LED_5: R11.1, U1.21 (PA11)
- new net LED_6: R12.1, U1.22 (PA12)
- new net LED_Connection: R5.1, U1.13 (PA7)
- new net LED_Debug: R6.1, U1.14 (PB0)
- new net LED_Error: R7.1, U1.15 (PB1)
- new net LED_emstop: R13.1, U1.30 (PB7)
- new net MCU_RST: C6.1, SW1.2, U1.4 (NRST)
- new net MCU_SWCLK: J5.2 (Pin_2), U1.24 (PA14)
- new net MCU_SWDIO: J5.4 (Pin_4), U1.23 (PA13)
- new net RF_BOOT: TP3.1, U2.24 (PB13~{})
- new net RF_LED: D2.1 (K), U2.11 (PB5)
- new net RF_RST: C4.1, SW2.2, U2.17 (RST)
- new net RF_SWCLK: TP2.1, U2.4 (PA14)
- new net RF_SWDIO: TP1.1, U2.3 (PA13)
- new net USART1_RX: J6.1 (Pin_1), U1.20 (PA10)
- new net USART1_TX: J6.3 (Pin_3), U1.19 (PA9)
- new net USART2_RX: U1.9 (PA3), U2.10 (PB6)
- new net USART2_TX: U1.8 (PA2), U2.9 (PB7)
- new net bustop: J4.1 (Pin_1), U1.29 (PB6)
- no-connect marks 0 -> 16
Other:
- note added: "Program Status"
