File: hardware/RemoteSwitchBoard/RemoteSwitchBoard.kicad_pcb (KiCad board)
At the start: 2 copper layers, 0 parts

Commit message: update
Parts:
- added BZ1: Buzzer, Buzzer_Beeper:Buzzer_TDK_PS1240P02BT_D12.2mm_H6.5mm, F.Cu at (70.8, 108.1)
- added C1: 0.1u, Capacitor_SMD:C_0603_1608Metric_Pad1.08x0.95mm_HandSolder, F.Cu at (93.8, 101.0)
- added C2: 0.1u, Capacitor_SMD:C_0603_1608Metric_Pad1.08x0.95mm_HandSolder, F.Cu at (96.3, 101.0)
- added C3: 4.7u, Capacitor_SMD:C_0603_1608Metric_Pad1.08x0.95mm_HandSolder, F.Cu at (98.8, 101.0)
- added C4: 0.1u, Capacitor_SMD:C_0603_1608Metric_Pad1.08x0.95mm_HandSolder, F.Cu at (118.1, 94.0)
- added C5: 4.7u, Capacitor_SMD:C_0603_1608Metric_Pad1.08x0.95mm_HandSolder, F.Cu at (103.1, 95.7)
- added C6: 0.1u, Capacitor_SMD:C_0603_1608Metric_Pad1.08x0.95mm_HandSolder, F.Cu at (76.1, 112.2)
- added C7: 10u, Capacitor_SMD:C_0603_1608Metric_Pad1.08x0.95mm_HandSolder, F.Cu at (108.8, 115.3)
- added C8: 22u, Capacitor_SMD:C_0603_1608Metric_Pad1.08x0.95mm_HandSolder, F.Cu at (110.9, 110.8)
- added D1: D, Diode_SMD:Nexperia_CFP3_SOD-123W, F.Cu at (111.2, 114.1)
- added D2: LED, LED_SMD:LED_0603_1608Metric_Pad1.05x0.95mm_HandSolder, F.Cu at (112.2, 108.5)
- added D4: LED, LED_SMD:LED_0603_1608Metric_Pad1.05x0.95mm_HandSolder, F.Cu at (114.3, 112.6)
- added D5: LED, LED_SMD:LED_0603_1608Metric_Pad1.05x0.95mm_HandSolder, F.Cu at (93.3, 108.8)
- added D6: LED, LED_SMD:LED_0603_1608Metric_Pad1.05x0.95mm_HandSolder, F.Cu at (93.3, 105.7)
- added D7: LED, LED_SMD:LED_0603_1608Metric_Pad1.05x0.95mm_HandSolder, F.Cu at (93.3, 110.4)
- added D9: LED, LED_SMD:LED_0603_1608Metric_Pad1.05x0.95mm_HandSolder, F.Cu at (93.4, 113.7)
- added H1: MountingHole, MountingHole:MountingHole_3.2mm_M3, F.Cu at (67.8, 87.0)
- added H2: MountingHole, MountingHole:MountingHole_3.2mm_M3, F.Cu at (123.9, 87.0)
- added H3: MountingHole, MountingHole:MountingHole_3.2mm_M3, F.Cu at (67.8, 126.1)
- added H4: MountingHole, MountingHole:MountingHole_3.2mm_M3, F.Cu at (123.9, 126.1)
- added J1: Conn_Coaxial, Connector_Coaxial:SMA_Molex_73251-2120_EdgeMount_Horizontal, F.Cu at (123.1, 104.1)
- added J10: XT30PW-M, Connector_AMASS:AMASS_XT30U-M_1x02_P5.0mm_Vertical, F.Cu at (124.5, 114.0)
- added J2: Conn_01x05, Connector_JST:JST_XH_B5B-XH-AM_1x05_P2.50mm_Vertical, F.Cu at (75.6, 127.1)
- added J3: Conn_01x02, Connector_JST:JST_XH_B2B-XH-A_1x02_P2.50mm_Vertical, F.Cu at (67.5, 93.5)
- added J4: Conn_01x02, Connector_JST:JST_XH_B2B-XH-A_1x02_P2.50mm_Vertical, F.Cu at (78.7, 94.5)
- added J5: Conn_01x04, Connector_JST:JST_XH_B4B-XH-A_1x04_P2.50mm_Vertical, F.Cu at (97.0, 88.1)
- added J6: Conn_01x04, Connector_JST:JST_XH_B4B-XH-A_1x04_P2.50mm_Vertical, F.Cu at (100.1, 106.7)
- added J7: Conn_01x02, Connector_JST:JST_XH_B2B-XH-A_1x02_P2.50mm_Vertical, F.Cu at (85.8, 107.7)
- added J8: Conn_01x05, Connector_JST:JST_XH_B5B-XH-AM_1x05_P2.50mm_Vertical, F.Cu at (74.6, 86.2)
- added J9: Conn_01x02, Connector_JST:JST_XH_B2B-XH-A_1x02_P2.50mm_Vertical, F.Cu at (67.1, 115.2)
- added R1: 10k, Capacitor_SMD:C_0603_1608Metric_Pad1.08x0.95mm_HandSolder, F.Cu at (84.5, 93.1)
- added R10: 1k, Capacitor_SMD:C_0603_1608Metric_Pad1.08x0.95mm_HandSolder, F.Cu at (81.4, 119.4)
- added R11: 1k, Capacitor_SMD:C_0603_1608Metric_Pad1.08x0.95mm_HandSolder, F.Cu at (81.4, 117.9)
- added R12: 1k, Capacitor_SMD:C_0603_1608Metric_Pad1.08x0.95mm_HandSolder, F.Cu at (81.4, 116.4)
- added R13: 1k, Capacitor_SMD:C_0603_1608Metric_Pad1.08x0.95mm_HandSolder, F.Cu at (68.3, 98.2)
- added R14: 1k, Capacitor_SMD:C_0603_1608Metric_Pad1.08x0.95mm_HandSolder, F.Cu at (85.8, 113.7)
- added R2: 1k, Capacitor_SMD:C_0603_1608Metric_Pad1.08x0.95mm_HandSolder, F.Cu at (115.6, 108.5)
- added R3: 1k, Capacitor_SMD:C_0603_1608Metric_Pad1.08x0.95mm_HandSolder, F.Cu at (81.4, 114.8)
- added R4: 1k, Capacitor_SMD:C_0603_1608Metric_Pad1.08x0.95mm_HandSolder, F.Cu at (114.4, 110.8)
- added R5: 1k, Capacitor_SMD:C_0603_1608Metric_Pad1.08x0.95mm_HandSolder, F.Cu at (93.3, 107.2)
- added R6: 1k, Capacitor_SMD:C_0603_1608Metric_Pad1.08x0.95mm_HandSolder, F.Cu at (93.3, 104.2)
- added R7: 1k, Capacitor_SMD:C_0603_1608Metric_Pad1.08x0.95mm_HandSolder, F.Cu at (93.4, 112.0)
- added R9: 1k, Capacitor_SMD:C_0603_1608Metric_Pad1.08x0.95mm_HandSolder, F.Cu at (93.3, 115.2)
- added SW1: SW_Push, GN10_Parts:TVAF, F.Cu at (79.2, 110.2)
- added SW2: SW_Push, GN10_Parts:TVAF, F.Cu at (120.9, 93.8)
- added TP1: TestPoint, TestPoint:TestPoint_Pad_D1.5mm, F.Cu at (116.0, 128.2)
- added TP2: TestPoint, TestPoint:TestPoint_Pad_D1.5mm, F.Cu at (118.8, 128.2)
- added TP3: TestPoint, TestPoint:TestPoint_Pad_D1.5mm, F.Cu at (113.2, 128.2)
- added U1: STM32F303K8Tx, Package_QFP:LQFP-32_7x7mm_P0.8mm, F.Cu at (87.7, 99.1)
- added U2: Wio-E5, GN10_Parts:LoRa-E5, F.Cu at (111.2, 100.2)
- added U4: AZ1117-3.3, Package_TO_SOT_SMD:SOT-223, F.Cu at (116.8, 117.3)
- added Y1: Crystal_GND2, Crystal:Resonator_SMD_Murata_CSTxExxV-3Pin_3.0x1.1mm_HandSoldering, F.Cu at (79.2, 104.8)
Routing:
- net +3.3V: track 0.00 -> 136.5 mm, vias 0 -> 2
- net USART2_RX: track 0.00 -> 51.0 mm, vias 0 -> 2
- net RF_BOOT: track 0.00 -> 40.3 mm, vias 0 -> 2
- net RF_SWDIO: track 0.00 -> 39.0 mm
- net LED_4: track 0.00 -> 38.9 mm, vias 0 -> 2
- net LED_5: track 0.00 -> 38.8 mm, vias 0 -> 2
- net USART2_TX: track 0.00 -> 37.3 mm, vias 0 -> 2
- net RF_SWCLK: track 0.00 -> 35.5 mm
- net emstop: track 0.00 -> 34.5 mm, vias 0 -> 2
- net LED_6: track 0.00 -> 28.6 mm, vias 0 -> 2
- net MCU_RST: track 0.00 -> 23.8 mm, vias 0 -> 2
- net LED_2: track 0.00 -> 21.8 mm, vias 0 -> 2
- net Net-(J2-Pin_3): track 0.00 -> 20.8 mm
- net +BATT: track 0.00 -> 20.6 mm
- net LED_emstop: track 0.00 -> 19.5 mm, vias 0 -> 2
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- added copper zone on B.Cu, net GND
- added copper zone on F.Cu, net GND
Other:
- board outline added: 64 x 47 mm
