File: hardware/ConsoleBoard/ConsoleBoard.kicad_pcb (KiCad board)
At the start: 2 copper layers, 80 x 25 mm, 26 parts, among them J2 Conn_01x05, J3 Conn_01x02, J4 Conn_01x02, J7 Conn_01x02, J8 Conn_01x05, Q1 AO3400A, SW1 SW_Push, SW3 SW_DIP_x04

Commit message: update
Parts:
- moved J8 1.59 mm to (106.7, 37.6)
- moved SW3 1.59 mm to (99.4, 27.9)
Routing:
- net +3.3V: track 49.9 -> 51.6 mm
- net Net-(D10-A): track 67.9 -> 69.3 mm
- net Net-(D10-K): track 82.6 -> 83.8 mm
