File: hardware/PowerCutoffBoard1/PowerCutoffBoard1.kicad_sch (KiCad schematic)
At the start: 47 parts, among them J1 Conn_Coaxial, J2 Conn_01x03, J3 Conn_01x04, J4 Conn_01x04, J5 Conn_01x04, J6 Conn_01x04, SW1 SW_Push, SW2 SW_Push, SW3 SW_DIP_x04, U1 STM32F303K8Tx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

Commit message: update
Parts:
- removed C12, C14: 10u, Capacitor_SMD:C_0805_2012Metric_Pad1.18x1.45mm_HandSolder, symbol Device:C
- removed J4: Conn_01x04, Connector_JST:JST_XH_S4B-XH-A_1x04_P2.50mm_Horizontal, symbol Connector_Generic:Conn_01x04
- added R3: 120, Resistor_SMD:R_0603_1608Metric_Pad0.98x0.95mm_HandSolder, symbol Device:R
- added Y1: Crystal_GND2, Crystal:Resonator_SMD_Murata_CSTxExxV-3Pin_3.0x1.1mm_HandSoldering, symbol Device:Crystal_GND2
Connections:
- net CAN_RX is gone; now on net CANRX: U1.21 (PA11)
- net CAN_TX is gone; now on net CANTX: U1.22 (PA12)
- net CANH: now also R3.1
- net CANL: now also R3.2
- net GND: now also Y1.2
- net USART1_RX: now also J6.1 (Pin_1); no longer U2.10 (PB6)
- net USART1_TX: now also J6.3 (Pin_3); no longer U2.9 (PB7)
- net USART2_RX: now also U2.10 (PB6); no longer J6.1 (Pin_1)
- net USART2_TX: now also U2.9 (PB7); no longer J6.3 (Pin_3)
- net at U1.2 (PF0): now also Y1.1
- net at U1.3 (PF1): now also Y1.3
- no-connect marks 17 -> 15
Other:
- moved on the sheet: R1

Commit message: fix:schematic
Connections:
- net DIP_1: now also U1.28 (PB5)
- net DIP_2: now also U1.27 (PB4)
- net DIP_3: now also U1.26 (PB3)
- net DIP_4: now also U1.25 (PA15)
- net IN_A: now also U1.29 (PB6)
- net IN_B: now also U1.30 (PB7)
- net LED_1: now also U1.12 (PA6)
- net LED_2: now also U1.11 (PA5)
- net LED_Connection: now also U1.13 (PA7)
- net LED_Debug: now also U1.14 (PB0)
- net LED_Error: now also U1.15 (PB1)
- no-connect marks 15 -> 19
Other:
- moved on the sheet: R1, Y1

Commit message: Wired PowerCutoffBoard1
Parts:
- added H1, H2, H3, H4: MountingHole, MountingHole:MountingHole_3.2mm_M3, symbol Mechanical:MountingHole

Commit message: update
Parts:
- removed Y1: Crystal_GND2, Crystal:Resonator_SMD_Murata_CSTxExxV-3Pin_3.0x1.1mm_HandSoldering, symbol Device:Crystal_GND2
Changed lines of the file:
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@@
 	(wire
 		(pts
-			(xy 118.11 144.78) (xy 130.81 144.78)
-		)
-		(stroke
-			(width 0)
-			(type default)
-		)
-	)
-	(wire
-		(pts
 			(xy 218.44 149.86) (xy 201.93 149.86)
 		)
@@
 	(wire
 		(pts
-			(xy 130.81 142.24) (xy 110.49 142.24)
-		)
-		(stroke
-			(width 0)
-			(type default)
-		)
-	)
-	(wire
-		(pts
 			(xy 125.73 33.02) (xy 137.16 33.02)
 		)
@@
 	(wire
 		(pts
-			(xy 110.49 142.24) (xy 110.49 144.78)
-		)
-		(stroke
-			(width 0)
-			(type default)
-		)
-	)
-	(wire
-		(pts
 			(xy 113.03 109.22) (xy 113.03 118.11)
 		)
@@
 	(symbol
 		(lib_id "power:GND")
-		(at 114.3 149.86 0)
-		(unit 1)
-		(exclude_from_sim no)
-		(in_bom yes)
-		(on_board yes)
-		(dnp no)
-		(fields_autoplaced yes)
-		(property "Reference" "#PWR017"
-			(at 114.3 156.21 0)
-			(effects
-				(font
-					(size 1.27 1.27)
-				)
-				(hide yes)
-			)
-		)
-		(property "Value" "GND"
-			(at 114.3 154.94 0)
-			(effects
-				(font
-					(size 1.27 1.27)
-				)
-			)
-		)
-		(property "Footprint" ""
-			(at 114.3 149.86 0)
-			(effects
-				(font
-					(size 1.27 1.27)
-				)
-				(hide yes)
-			)
-		)
-		(property "Datasheet" ""
-			(at 114.3 149.86 0)
-			(effects
-				(font
-					(size 1.27 1.27)
-				)
-				(hide yes)
-			)
-		)
-		(property "Description" "Power symbol creates a global label with name \"GND\" , ground"
-			(at 114.3 149.86 0)
-			(effects
-				(font
-					(size 1.27 1.27)
-				)
-				(hide yes)
-			)
-		)
-		(pin "1"
-		)
-		(instances
-			(project "PowerCutoffBoard1"
-				(path "/f159c84c-1623-42a3-b839-f1b33ec92c24"
-					(reference "#PWR017")
-					(unit 1)
-				)
-			)
-		)
-	)
-	(symbol
-		(lib_id "power:GND")
 		(at 66.04 137.16 90)
 		(unit 1)
@@
 					(unit 1)
 				)
-			)
-		)
-	)
-	(symbol
-		(lib_id "Device:Crystal_GND2")
-		(at 114.3 144.78 0)
-		(unit 1)
-		(exclude_from_sim no)
-		(in_bom yes)
-		(on_board yes)
-		(dnp no)
-		(fields_autoplaced yes)
-		(property "Reference" "Y1"
-			(at 114.3 137.16 0)
-			(effects
-				(font
-					(size 1.27 1.27)
-				)
-			)
-		)
-		(property "Value" "Crystal_GND2"
-			(at 114.3 139.7 0)
-			(effects
-				(font
-					(size 1.27 1.27)
-				)
-			)
-		)
-		(property "Footprint" "Crystal:Resonator_SMD_Murata_CSTxExxV-3Pin_3.0x1.1mm_HandSoldering"
-			(at 114.3 144.78 0)
-			(effects
-				(font
-					(size 1.27 1.27)
-				)
-				(hide yes)
-			)
-		)
-		(property "Datasheet" "~"
-			(at 114.3 144.78 0)
-			(effects
-				(font
-					(size 1.27 1.27)
-				)
-				(hide yes)
-			)
-		)
-		(property "Description" "Three pin crystal, GND on pin 2"
-			(at 114.3 144.78 0)
-			(effects
-				(font
-					(size 1.27 1.27)
-				)
-				(hide yes)
-			)
-		)
-		(pin "3"
-		)
-		(pin "2"
-		)
-		(pin "1"
-		)
-		(instances
-			(project ""
-				(path "/f159c84c-1623-42a3-b839-f1b33ec92c24"
-					(reference "Y1")
-					(unit 1)
-				)

Commit message: update:取捨選択とノイズ対策
Parts:
- removed TP1, TP2, TP3: TestPoint, TestPoint:TestPoint_Pad_D1.5mm, symbol Connector:TestPoint
Connections:
- no-connect marks 19 -> 21
