File: hardware/PowerCutoffBoard1/PowerCutoffBoard1.kicad_pcb (KiCad board)
At the start: 2 copper layers, 50 x 45 mm, 50 parts, among them J1 Conn_Coaxial, J2 Conn_01x03, J3 Conn_01x04, J5 Conn_01x04, J6 Conn_01x04, SW1 SW_Push, SW2 SW_Push, SW3 SW_DIP_x04, U1 STM32F303K8Tx, U2 Wio-E5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

Commit message: update
Parts:
- removed Y1: Crystal_GND2, Crystal:Resonator_SMD_Murata_CSTxExxV-3Pin_3.0x1.1mm_HandSoldering
Connections:
- U1 pad 2: Net-(U1-PF0) -> unconnected-(U1-PF0-Pad2)
- U1 pad 3: Net-(U1-PF1) -> unconnected-(U1-PF1-Pad3)
Routing:
- net Net-(U1-PF1): track 4.11 -> 0.00 mm
- net Net-(U1-PF0): track 4.03 -> 0.00 mm
- net +3.3V: track 142.4 -> 140.8 mm, vias 0 -> 2
- net GND: vias 26 -> 38

Commit message: update
Routing:
- net GND: vias 38 -> 53
Changed lines of the file:
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@@
+	)
+	(via
+		(at 167.2 110.94)
+		(size 0.8)
+		(drill 0.4)
+		(layers "F.Cu" "B.Cu")
+		(free yes)
+		(net 1)
 	)
 	(via
@@
 	)
 	(via
+		(at 171.2 120.82)
+		(size 0.8)
+		(drill 0.4)
+		(layers "F.Cu" "B.Cu")
+		(free yes)
+		(net 1)
+	)
+	(via
 		(at 185.55 115.6)
 		(size 0.8)
@@
 	)
 	(via
+		(at 175.39 122.22)
+		(size 0.8)
+		(drill 0.4)
+		(layers "F.Cu" "B.Cu")
+		(free yes)
+		(net 1)
+	)
+	(via
+		(at 186.45 141.28)
+		(size 0.8)
+		(drill 0.4)
+		(layers "F.Cu" "B.Cu")
+		(free yes)
+		(net 1)
+	)
+	(via
 		(at 157.06 114.13)
 		(size 0.8)
@@
 	)
 	(via
+		(at 165.65 149.3)
+		(size 0.8)
+		(drill 0.4)
+		(layers "F.Cu" "B.Cu")
+		(free yes)
+		(net 1)
+	)
+	(via
 		(at 176.3 138.575)
 		(size 0.8)
@@
 	)
 	(via
+		(at 155.22 129.65)
+		(size 0.8)
+		(drill 0.4)
+		(layers "F.Cu" "B.Cu")
+		(free yes)
+		(net 1)
+	)
+	(via
 		(at 150.7 119.3)
 		(size 0.8)
@@
 	)
 	(via
+		(at 182.23 134.88)
+		(size 0.8)
+		(drill 0.4)
+		(layers "F.Cu" "B.Cu")
+		(free yes)
+		(net 1)
+	)
+	(via
 		(at 151.875 129.875)
 		(size 0.8)
@@
 	)
 	(via
+		(at 175.6 149.3)
+		(size 0.8)
+		(drill 0.4)
+		(layers "F.Cu" "B.Cu")
+		(free yes)
+		(net 1)
+	)
+	(via
 		(at 177.25 138.8)
 		(size 0.8)
@@
 	)
 	(via
+		(at 154.82 134.39)
+		(size 0.8)
+		(drill 0.4)
+		(layers "F.Cu" "B.Cu")
+		(free yes)
+		(net 1)
+	)
+	(via
+		(at 175.07 118.72)
+		(size 0.8)
+		(drill 0.4)
+		(layers "F.Cu" "B.Cu")
+		(free yes)
+		(net 1)
+	)
+	(via
 		(at 164.49 123.37)
 		(size 0.8)
@@
 	)
 	(via
+		(at 165.07 110.22)
+		(size 0.8)
+		(drill 0.4)
+		(layers "F.Cu" "B.Cu")
+		(free yes)
+		(net 1)
+	)
+	(via
 		(at 172.05 114.06)
 		(size 0.8)
@@
 	)
 	(via
+		(at 178.63 134.71)
+		(size 0.8)
+		(drill 0.4)
+		(layers "F.Cu" "B.Cu")
+		(free yes)
+		(net 1)
+	)
+	(via
+		(at 165.12 111.13)
+		(size 0.8)
+		(drill 0.4)
+		(layers "F.Cu" "B.Cu")
+		(free yes)
+		(net 1)
+	)
+	(via
+		(at 167.18 110.08)
+		(size 0.8)
+		(drill 0.4)
+		(layers "F.Cu" "B.Cu")
+		(free yes)
+		(net 1)
+	)
+	(via
 		(at 195.92 121.5)
 		(size 0.8)
@@
 		(size 0.8)
 		(drill 0.4)
+		(layers "F.Cu" "B.Cu")
+		(free yes)
+		(net 1)
+	)
+	(via
+		(at 177.85 130.74)
+		(size 0.8)
+		(drill 0.4)

Commit message: update
Routing:
- net +5V: track 61.3 -> 61.9 mm
Changed lines of the file:
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@@
 	)
 	(segment
-		(start 191.78 108.1135)
-		(end 191.78 116.067)
-		(width 0.25)
+		(start 178.22 123.79)
+		(end 177.1385 122.7085)
+		(width 0.6)
 		(layer "F.Cu")
 		(net 36)
 	)
 	(segment
-		(start 184.07 107.555)
-		(end 183.9 107.725)
-		(width 0.25)
+		(start 190.754 107.0875)
+		(end 188.9465 107.0875)
+		(width 0.6)
+		(layer "F.Cu")
+		(net 36)
+	)
+	(segment
+		(start 190.754 107.0875)
+		(end 191.955 108.2885)
+		(width 0.6)
+		(layer "F.Cu")
+		(net 36)
+	)
+	(segment
+		(start 184.085 107.555)
+		(end 183.98 107.66)
+		(width 0.6)
+		(layer "F.Cu")
+		(net 36)
+	)
+	(segment
+		(start 191.955 118.844)
+		(end 191.955 123.286002)
+		(width 0.6)
+		(layer "F.Cu")
+		(net 36)
+	)
+	(segment
+		(start 186.944 127.508)
+		(end 186.944 129.286)
+		(width 0.6)
+		(layer "F.Cu")
+		(net 36)
+	)
+	(segment
+		(start 186.654 107.185)
+		(end 186.284 107.555)
+		(width 0.6)
 		(layer "F.Cu")
 		(net 36)
@@
 		(start 188.9465 107.0875)
 		(end 188.849 107.185)
-		(width 0.25)
+		(width 0.6)
 		(layer "F.Cu")
 		(net 36)
 	)
 	(segment
-		(start 186.944 127.508)
-		(end 186.944 129.286)
-		(width 0.25)
+		(start 186.944 129.286)
+		(end 186.944 131.637)
+		(width 0.6)
 		(layer "F.Cu")
 		(net 36)
 	)
 	(segment
-		(start 188.71 107.185)
-		(end 188.34 107.555)
-		(width 0.25)
+		(start 188.849 107.185)
+		(end 186.654 107.185)
+		(width 0.6)
 		(layer "F.Cu")
 		(net 36)
 	)
 	(segment
-		(start 190.754 107.0875)
-		(end 191.78 108.1135)
-		(width 0.25)
+		(start 191.955 108.2885)
+		(end 191.955 115.892)
+		(width 0.6)
 		(layer "F.Cu")
 		(net 36)
 	)
 	(segment
-		(start 190.754 107.0875)
-		(end 188.9465 107.0875)
-		(width 0.25)
-		(layer "F.Cu")
-		(net 36)
-	)
-	(segment
-		(start 188.34 107.555)
-		(end 186.284 107.555)
-		(width 0.25)
-		(layer "F.Cu")
-		(net 36)
-	)
-	(segment
-		(start 178.125 123.725)
-		(end 177.1385 122.7385)
-		(width 0.25)
-		(layer "F.Cu")
-		(net 36)
-	)
-	(segment
-		(start 187.485514 127.508)
-		(end 191.78 123.213514)
-		(width 0.25)
-		(layer "F.Cu")
-		(net 36)
-	)
-	(segment
-		(start 191.78 116.067)
+		(start 191.955 115.892)
 		(end 190.479 117.368)
-		(width 0.25)
-		(layer "F.Cu")
-		(net 36)
-	)
-	(segment
-		(start 177.1385 122.7385)
-		(end 177.1385 120.65)
-		(width 0.25)
-		(layer "F.Cu")
-		(net 36)
-	)
-	(segment
-		(start 191.78 118.669)
-		(end 190.479 117.368)
-		(width 0.25)
-		(layer "F.Cu")
-		(net 36)
-	)
-	(segment
-		(start 191.78 123.213514)
-		(end 191.78 118.669)
-		(width 0.25)
+		(width 0.6)
 		(layer "F.Cu")
 		(net 36)
@@
 	(segment
 		(start 186.284 107.555)
-		(end 184.07 107.555)
-		(width 0.25)
+		(end 184.085 107.555)
+		(width 0.6)
 		(layer "F.Cu")
 		(net 36)
 	)
 	(segment
-		(start 188.849 107.185)
-		(end 188.71 107.185)
-		(width 0.25)
+		(start 177.1385 122.7085)
+		(end 177.1385 120.65)
+		(width 0.6)
 		(layer "F.Cu")
 		(net 36)
 	)
 	(segment
-		(start 186.944 127.508)
-		(end 187.485514 127.508)
-		(width 0.25)
+		(start 190.479 117.368)
+		(end 191.955 118.844)
+		(width 0.6)
 		(layer "F.Cu")
 		(net 36)
 	)
 	(segment
-		(start 179.262 120.65)
-		(end 177.1385 120.65)
-		(width 0.25)
+		(start 191.955 123.286002)
+		(end 187.733002 127.508)
+		(width 0.6)
 		(layer "F.Cu")
 		(net 36)
 	)
 	(segment
-		(start 186.944 131.637)
-		(end 186.944 129.286)
-		(width 0.25)
+		(start 177.1385 120.65)
+		(end 179.262 120.65)
+		(width 0.6)
+		(layer "F.Cu")
+		(net 36)
+	)
+	(segment
+		(start 187.733002 127.508)
+		(end 186.944 127.508)
+		(width 0.6)
 		(layer "F.Cu")
 		(net 36)
 	)
 	(via
-		(at 183.9 107.725)
-		(size 0.8)
-		(drill 0.4)
+		(at 178.22 123.79)
+		(size 1)
+		(drill 0.7)
 		(layers "F.Cu" "B.Cu")
 		(net 36)
 	)
 	(via
-		(at 178.125 123.725)
-		(size 0.8)
-		(drill 0.4)
+		(at 183.98 107.66)
+		(size 1)
+		(drill 0.7)
 		(layers "F.Cu" "B.Cu")
 		(net 36)
 	)
 	(segment
-		(start 183.9 107.725)
-		(end 183.9 121.1)
-		(width 0.25)
+		(start 183.98 107.66)
+		(end 183.87 107.77)
+		(width 0.6)
 		(layer "B.Cu")
 		(net 36)
 	)
 	(segment
-		(start 181.275 123.725)
-		(end 178.125 123.725)
-		(width 0.25)
+		(start 183.87 121.01)
+		(end 183.87 121.22)
+		(width 0.6)
 		(layer "B.Cu")
 		(net 36)
 	)
 	(segment
-		(start 183.9 121.1)
-		(end 181.275 123.725)
-		(width 0.25)
+		(start 183.87 107.77)
+		(end 183.87 121.01)
+		(width 0.6)
 		(layer "B.Cu")
 		(net 36)
+	)
+	(segment
+		(start 183.87 121.22)
+		(end 181.38 123.71)
+		(width 0.6)
+		(layer "B.Cu")
+		(net 36)
+	)
+	(segment
+		(start 181.38 123.71)
+		(end 181.3 123.79)
+		(width 0.6)
+		(layer "B.Cu")
+		(net 36)
+	)
+	(segment
+		(start 181.3 123.79)
+		(end 178.22 123.79)
+		(width 0.6)
+		(layer "B.Cu")
+		(net 36)

Commit message: update
Routing:
- net GND: vias 53 -> 59
Changed lines of the file:
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@@
+	)
+	(via
+		(at 173.53 125.19)
+		(size 0.8)
+		(drill 0.4)
+		(layers "F.Cu" "B.Cu")
+		(free yes)
+		(net 1)
 	)
 	(via
@@
 	)
 	(via
+		(at 157 124.96)
+		(size 0.8)
+		(drill 0.4)
+		(layers "F.Cu" "B.Cu")
+		(free yes)
+		(net 1)
+	)
+	(via
 		(at 185.55 115.6)
 		(size 0.8)
@@
 	)
 	(via
+		(at 181.56 126.69)
+		(size 0.8)
+		(drill 0.4)
+		(layers "F.Cu" "B.Cu")
+		(free yes)
+		(net 1)
+	)
+	(via
+		(at 155.46 132.07)
+		(size 0.8)
+		(drill 0.4)
+		(layers "F.Cu" "B.Cu")
+		(free yes)
+		(net 1)
+	)
+	(via
 		(at 175.39 122.22)
 		(size 0.8)
@@
 	)
 	(via
+		(at 159.95 126.89)
+		(size 0.8)
+		(drill 0.4)
+		(layers "F.Cu" "B.Cu")
+		(free yes)
+		(net 1)
+	)
+	(via
 		(at 165.65 149.3)
 		(size 0.8)
@@
 		(size 0.8)
 		(drill 0.4)
+		(layers "F.Cu" "B.Cu")
+		(free yes)
+		(net 1)
+	)
+	(via
+		(at 172.05 141.78)
+		(size 0.8)
+		(drill 0.4)

Commit message: update:取捨選択とノイズ対策
Parts:
- removed TP1, TP2, TP3: TestPoint, TestPoint:TestPoint_Pad_D1.5mm
- moved R1 1.04 mm to (174.9, 139.7), turned to 0 degrees
Routing:
- net RF_SWCLK: track 20.3 -> 0.00 mm
- net RF_BOOT: track 15.3 -> 0.00 mm
- net RF_SWDIO: track 15.1 -> 0.00 mm
- net USART2_RX: track 16.2 -> 12.7 mm
- net RF_RST: track 19.8 -> 23.1 mm
- net IN_B: track 20.4 -> 17.9 mm
- net +5V: track 61.9 -> 60.7 mm
- net DIP_2: track 16.2 -> 15.2 mm
- net CANTX: track 27.3 -> 27.9 mm
- net GND: vias 59 -> 82
Other:
- board text added: "3.3 CLK GND DIO"
- board text added: "CH-bit1"
- board text added: "CH-bit2"
- board text added: "CONN"
- board text added: "DEBUG"
- board text added: "ERROR"
- board text added: "POWER"
- board text added: "RF_LED"
- board text added: "RF_RST"
- board text added: "RX 3.3 TX GND"

Commit message: fix
Parts:
- moved C2 1.47 mm to (157.3, 129.5)
- moved C5 1.41 mm to (157.3, 127.9)
Routing:
- net +3.3V: track 140.8 -> 139.1 mm
- net GND: vias 82 -> 83
Changed lines of the file:
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@@
 			(outputformat 1)
 			(mirror no)
-			(drillshape 1)
+			(drillshape 0)
 			(scaleselection 1)
-			(outputdirectory "")
+			(outputdirectory "PowerCutoffBoard1/")
 		)
 	)
@@
 	(footprint "Capacitor_SMD:C_0603_1608Metric_Pad1.08x0.95mm_HandSolder"
 		(layer "F.Cu")
-		(at 156.2 128.525 180)
+		(at 157.3 129.5 180)
 		(descr "Capacitor SMD 0603 (1608 Metric), square (rectangular) end terminal, IPC_7351 nominal with elongated pad for handsoldering. (Body size source: IPC-SM-782 page 76, https://www.pcb-3d.com/wordpress/wp-content/uploads/ipc-sm-782a_amendment_1_and_2.pdf), generated with kicad-footprint-generator")
 		(tags "capacitor handsolder")
 		(property "Reference" "C2"
-			(at 0 1.45 0)
+			(at -2.8 0 0)
 			(layer "F.SilkS")
 			(effects
@@
 		(tags "capacitor handsolder")
 		(property "Reference" "R1"
-			(at 0 -1.43 0)
+			(at 1.4945 -1.6 0)
 			(layer "F.SilkS")
 			(effects
@@
 		(tags "CFP3 SOD-123W")
 		(property "Reference" "D1"
-			(at 0 -2 90)
+			(at 2.25 -1.951 90)
 			(layer "F.SilkS")
 			(effects
@@
 		(tags "capacitor handsolder")
 		(property "Reference" "C7"
-			(at 0 -1.43 90)
+			(at 2.95 -1.546 90)
 			(layer "F.SilkS")
 			(effects
@@
 		(tags "LQFP QFP")
 		(property "Reference" "U1"
-			(at 0 -5.88 0)
+			(at 1.085 -6.15 0)
 			(layer "F.SilkS")
 			(effects
@@
 	(footprint "Capacitor_SMD:C_0603_1608Metric_Pad1.08x0.95mm_HandSolder"
 		(layer "F.Cu")
-		(at 156.2125 126.975 180)
+		(at 157.3 127.87 180)
 		(descr "Capacitor SMD 0603 (1608 Metric), square (rectangular) end terminal, IPC_7351 nominal with elongated pad for handsoldering. (Body size source: IPC-SM-782 page 76, https://www.pcb-3d.com/wordpress/wp-content/uploads/ipc-sm-782a_amendment_1_and_2.pdf), generated with kicad-footprint-generator")
 		(tags "capacitor handsolder")
 		(property "Reference" "C5"
-			(at 0 -1.43 0)
+			(at -2.8 -0.13 0)
 			(layer "F.SilkS")
 			(effects
@@
 	)
 	(via
+		(at 177.9 126.6)
+		(size 0.8)
+		(drill 0.4)
+		(layers "F.Cu" "B.Cu")
+		(free yes)
+		(net 1)
+	)
+	(via
 		(at 151.384 131.064)
 		(size 0.8)
@@
 	)
 	(segment
-		(start 157.075 126.975)
-		(end 157.075 128.5125)
-		(width 0.4)
-		(layer "F.Cu")
-		(net 2)
-	)
-	(segment
 		(start 161.036 148.463)
 		(end 159.766 148.463)
@@
 	)
 	(segment
-		(start 157.83 127.73)
-		(end 157.075 126.975)
-		(width 0.4)
-		(layer "F.Cu")
-		(net 2)
-	)
-	(segment
 		(start 188.719 109.855)
 		(end 188.849 109.985)
@@
 	)
 	(segment
-		(start 157.088 126.975)
-		(end 158.683 125.38)
+		(start 158.1625 129.5)
+		(end 158.1625 125.9005)
 		(width 0.4)
 		(layer "F.Cu")
@@
 	)
 	(segment
-		(start 157.075 126.975)
-		(end 157.088 126.975)
-		(width 0.4)
-		(layer "F.Cu")
-		(net 2)
-	)
-	(segment
 		(start 191.437 145.516819)
 		(end 191.437 146.803181)
@@
 	)
 	(segment
-		(start 159.01 127.73)
-		(end 157.83 127.73)
-		(width 0.4)
-		(layer "F.Cu")
-		(net 2)
-	)
-	(segment
 		(start 184.3915 125.4)
 		(end 184.3915 123.712)
@@
 	)
 	(segment
-		(start 167.91 130.55)
-		(end 167.04 130.55)
+		(start 159.2 129.5)
+		(end 158.1625 129.5)
 		(width 0.4)
 		(layer "F.Cu")
@@
 	)
 	(segment
-		(start 157.075 128.5125)
-		(end 157.0625 128.525)
+		(start 167.91 130.55)
+		(end 167.04 130.55)
 		(width 0.4)
 		(layer "F.Cu")
@@
 	)
 	(segment
+		(start 158.1625 125.9005)
+		(end 158.683 125.38)
+		(width 0.4)
+		(layer "F.Cu")
+		(net 2)
+	)
+	(segment
 		(start 190.704181 147.536)
 		(end 184.062 147.536)
@@
 	)
 	(via
-		(at 159.01 127.73)
+		(at 159.2 129.5)
 		(size 0.8)
 		(drill 0.4)
@@
 	)
 	(segment
-		(start 166.32 131.27)
-		(end 162.55 131.27)
+		(start 160.97 131.27)
+		(end 166.32 131.27)
 		(width 0.4)
 		(layer "B.Cu")
@@
 	)
 	(segment
-		(start 162.55 131.27)
-		(end 159.01 127.73)
+		(start 159.2 129.5)
+		(end 160.97 131.27)
 		(width 0.4)
 		(layer "B.Cu")
